File: greyhound_probe.kicad_sch (KiCad schematic)
At the start: 40 parts, among them J1 USB_C_Receptacle_USB2.0, J2 Conn_01x04_Male, J3 FTSH-105-01-L-DV-K-TR, Q1 IRLML6401, SW1 SW_SPDT, U1 XC6206P332MR, U2 USBLC6-2SC6, U3 STM32F072CBUx

Commit message: Better spacing of a few signal traces and vias
Parts:
- C1, C2, C7: LCSC Part (none) -> C1592
- C10, C11, C3, C5, C6: LCSC Part (none) -> C66501
- C4, C9: LCSC Part (none) -> C8032
- C8: LCSC Part (none) -> C1589
- J2: LCSC Part (none) -> C2935910
- R10, R11, R9: LCSC Part (none) -> C105588
- R3: LCSC Part (none) -> C105428
- R5, R6, R7: LCSC Part (none) -> C22548
- R8: LCSC Part (none) -> C99198
Changed lines of the file:
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@@
+      (effects (font (size 1.27 1.27)) hide)
+    )
+    (property "LCSC Part" "C105588" (id 5) (at 358.902 159.766 0)
       (effects (font (size 1.27 1.27)) hide)
     )
@@
     )
     (property "Datasheet" "~" (id 3) (at 139.8016 145.2372 0)
+      (effects (font (size 1.27 1.27)) hide)
+    )
+    (property "LCSC Part" "C66501" (id 5) (at 139.8016 145.2372 0)
       (effects (font (size 1.27 1.27)) hide)
     )
@@
       (effects (font (size 1.27 1.27)) hide)
     )
+    (property "LCSC Part" "C105588" (id 5) (at 358.902 162.306 0)
+      (effects (font (size 1.27 1.27)) hide)
+    )
     (pin "1")
     (pin "2")
@@
       (effects (font (size 1.27 1.27)) hide)
     )
-    (property "LCSC Part" "" (id 4) (at 226.0092 122.682 0)
+    (property "LCSC Part" "C22548" (id 4) (at 226.0092 122.682 0)
       (effects (font (size 1.27 1.27)) hide)
     )
@@
     )
     (property "Datasheet" "~" (id 3) (at 217.932 71.374 0)
+      (effects (font (size 1.27 1.27)) hide)
+    )
+    (property "LCSC Part" "C1589" (id 5) (at 217.932 71.374 0)
       (effects (font (size 1.27 1.27)) hide)
     )
@@
       (effects (font (size 1.27 1.27)) hide)
     )
+    (property "LCSC Part" "C66501" (id 5) (at 195.58 71.374 0)
+      (effects (font (size 1.27 1.27)) hide)
+    )
     (pin "1")
     (pin "2")
@@
     )
     (property "Datasheet" "~" (id 3) (at 190.754 71.374 0)
+      (effects (font (size 1.27 1.27)) hide)
+    )
+    (property "LCSC Part" "C8032" (id 5) (at 190.754 71.374 0)
       (effects (font (size 1.27 1.27)) hide)
     )
@@
       (effects (font (size 1.27 1.27)) hide)
     )
+    (property "LCSC Part" "C2935910" (id 4) (at 346.0496 155.1432 0)
+      (effects (font (size 1.27 1.27)) hide)
+    )
     (pin "1")
     (pin "2")
@@
       (effects (font (size 1.27 1.27)) hide)
     )
+    (property "LCSC Part" "C66501" (id 5) (at 233.172 71.374 0)
+      (effects (font (size 1.27 1.27)) hide)
+    )
     (pin "1")
     (pin "2")
@@
       (effects (font (size 1.27 1.27)) hide)
     )
-    (property "LCSC Part" "" (id 4) (at 215.3412 122.682 0)
+    (property "LCSC Part" "C22548" (id 4) (at 215.3412 122.682 0)
       (effects (font (size 1.27 1.27)) hide)
     )
@@
       (effects (font (size 1.27 1.27)) hide)
     )
+    (property "LCSC Part" "C1592" (id 5) (at 213.106 71.374 0)
+      (effects (font (size 1.27 1.27)) hide)
+    )
     (pin "1")
     (pin "2")
@@
       (effects (font (size 1.27 1.27)) hide)
     )
+    (property "LCSC Part" "C1592" (id 5) (at 37.846 127.508 0)
+      (effects (font (size 1.27 1.27)) hide)
+    )
     (pin "1")
     (pin "2")
@@
     )
     (property "Datasheet" "~" (id 3) (at 62.992 127.508 0)
+      (effects (font (size 1.27 1.27)) hide)
+    )
+    (property "LCSC Part" "C1592" (id 5) (at 62.992 127.508 0)
       (effects (font (size 1.27 1.27)) hide)
     )
@@
       (effects (font (size 1.27 1.27)) hide)
     )
-    (property "LCSC Part" "" (id 4) (at 132.08 137.16 0)
+    (property "LCSC Part" "C105428" (id 4) (at 132.08 137.16 0)
       (effects (font (size 1.27 1.27)) hide)
     )
@@
     )
     (property "Datasheet" "~" (id 3) (at 389.2296 108.1024 0)
+      (effects (font (size 1.27 1.27)) hide)
+    )
+    (property "LCSC Part" "C66501" (id 5) (at 389.2296 108.1024 0)
       (effects (font (size 1.27 1.27)) hide)
     )
@@
       (effects (font (size 1.27 1.27)) hide)
     )
+    (property "LCSC Part" "C105588" (id 5) (at 367.284 50.8508 0)
+      (effects (font (size 1.27 1.27)) hide)
+    )
     (pin "1")
     (pin "2")
@@
       (effects (font (size 1.27 1.27)) hide)
     )
+    (property "LCSC Part" "C99198" (id 4) (at 355.6 111.8108 0)
+      (effects (font (size 1.27 1.27)) hide)
+    )
     (pin "1")
     (pin "2")
@@
       (effects (font (size 1.27 1.27)) hide)
     )
-    (property "LCSC Part" "" (id 4) (at 204.9272 122.682 0)
+    (property "LCSC Part" "C22548" (id 4) (at 204.9272 122.682 0)
       (effects (font (size 1.27 1.27)) hide)
     )
@@
       (effects (font (size 1.27 1.27)) hide)
     )
+    (property "LCSC Part" "C8032" (id 5) (at 228.346 71.374 0)
+      (effects (font (size 1.27 1.27)) hide)
+    )
     (pin "1")
     (pin "2")
@@
       (effects (font (size 1.27 1.27)) hide)
     )
+    (property "LCSC Part" "C66501" (id 5) (at 202.946 71.374 0)
+      (effects (font (size 1.27 1.27)) hide)
+    )

Commit message: Added SWD, rearranged bottom part
Parts:
- removed H2: MountingHole, MountingHole:MountingHole_2.2mm_M2, symbol Mechanical:MountingHole
- added J4: Conn_01x02_Male, Connector_PinHeader_2.54mm:PinHeader_1x02_P2.54mm_Vertical, symbol Connector:Conn_01x02_Male
- renumbered R8 to R10, R9 to R8, R10 to R9
Connections:
- net SWDIO: now reaches U3.34 (PA13)
- net SWDIO: now also J4.1 (Pin_1)
- net SWCLK: now reaches U3.37 (PA14)
- net SWCLK: now also J4.2 (Pin_2)
- no-connect marks 26 -> 24
Other:
- note added: "SWD"
- note added: "Target JTAG/SWD"
- note removed: "JTAG/SWD"
- moved on the sheet: H3, H4, J2, R8, R9
