File: greyhound_probe.kicad_sch (KiCad schematic)
At the start: 40 parts, among them J1 USB_C_Receptacle_USB2.0, J2 Conn_01x04_Male, J3 FTSH-105-01-L-DV-K-TR, J4 Conn_01x02_Male, Q1 IRLML6401, SW1 SW_SPDT, U1 XC6206P332MR, U2 USBLC6-2SC6, U3 STM32F072CBUx

Commit message: Added in series resistor to mosfet gate, nrst pullup, more regulator caps, reduced via sharing
Parts:
- removed C11: 100nF, Capacitor_SMD:C_0603_1608Metric, symbol Device:C_Small
- added C1, C3: 4.7uF, Capacitor_SMD:C_0603_1608Metric, symbol Device:C_Small
- added R13: 10k, Resistor_SMD:R_0603_1608Metric, symbol Device:R_Small
- added R5: 1k, Resistor_SMD:R_0603_1608Metric, symbol Device:R_Small
- renumbered C8 to C10, C9 to C11, C10 to C12, C1 to C2, C2 to C4, C3 to C5, C4 to C6, C5 to C7, C6 to C8, C7 to C9, H3 to H1, H4 to H2, H1 to H3, R9 to R10, R10 to R11, R11 to R12, R5 to R6, R6 to R7, R7 to R8, R8 to R9
Connections:
- net +3.3V: now also C3.1, R13.1
- net GND: now also C1.2, C3.2
- net NRST: now also R13.2
- net TARGET_POWER: now also R5.2; no longer Q1.1 (G)
- net at C2.1, FB1.2, U1.3 (VI): now also C1.1
- new net: Q1.1 (G), R5.1
Other:
- moved on the sheet: C2, C4, F1, FB1, U1
